File: hardware/bells-theorem/panel.sch (KiCad schematic (older format))
At the start: 68 parts, among them J10 D, J11 C, J12 DA, J13 CD, J14 DAB, J15 CDA, J16 A, J17 B, J18 AB, J19 BC, J20 ABC, J21 BCD, J22 left, J23 right, J4 IN, J5 CVA, J6 CVB, J7 CVC, J8 CVD, J9 ABCD, Q1 Q_NPN_BCE, Q10 Q_NPN_BCE, Q12 Q_NPN_BCE, Q13 Q_NPN_BCE, Q3 Q_NPN_BCE, Q4 Q_NPN_BCE, Q6 Q_NPN_BCE, Q7 Q_NPN_BCE, Q9 Q_NPN_BCE, SW1 A, SW2 D, SW3 B, SW4 C

Commit message: take gerbers out of the repo, push latest updates
Parts:
- removed SW1: A, Rotary_Encoder:RotaryEncoder_Alps_EC12E-Switch_Vertical_H20mm_CircularMountingHoles, symbol device:Rotary_Encoder_Switch
- removed SW2: D, Rotary_Encoder:RotaryEncoder_Alps_EC12E-Switch_Vertical_H20mm_CircularMountingHoles, symbol device:Rotary_Encoder_Switch
- removed SW3: B, Rotary_Encoder:RotaryEncoder_Alps_EC12E-Switch_Vertical_H20mm_CircularMountingHoles, symbol device:Rotary_Encoder_Switch
- removed SW4: C, Rotary_Encoder:RotaryEncoder_Alps_EC12E-Switch_Vertical_H20mm_CircularMountingHoles, symbol device:Rotary_Encoder_Switch
- added Q11, Q2, Q5, Q8: 2N3904, Package_TO_SOT_SMD:SOT-23_Handsoldering, symbol device:Q_NPN_BEC
- added R100, R101: 470R, Resistor_SMD:R_0805_2012Metric_Pad1.15x1.40mm_HandSolder, symbol device:R_US
- added R102, R103, R93, R94, R95, R96, R97, R98, R99: 4.7K, Resistor_SMD:R_0805_2012Metric_Pad1.15x1.40mm_HandSolder, symbol device:R_US
- added R104: 15K, Resistor_SMD:R_0805_2012Metric_Pad1.15x1.40mm_HandSolder, symbol device:R_US
- added R105, R131: 390R, Resistor_SMD:R_0805_2012Metric_Pad1.15x1.40mm_HandSolder, symbol device:R_US
- added R92: 2.2K, Resistor_SMD:R_0805_2012Metric_Pad1.15x1.40mm_HandSolder, symbol device:R_US
- added S1, S2, S3, S4: ENCODER-RGB-SWITCH, My Library:ENCODER_LED_3_KIT, symbol petelib:ENCODER-RGB-SWITCH
- Q1, Q10, Q12, Q13, Q3, Q4, Q6, Q7, Q9: value Q_NPN_BCE -> 2N3904; symbol device:Q_NPN_BCE -> device:Q_NPN_BEC
- R7: value 4.7K -> 420R
- R8: value 4.7K -> 470R
Connections:
- net +12V: now also S1.5 (+)
- net +3V3: now also R94.1, R95.1, R96.1, R97.1, S2.5 (+), S3.5 (+), S4.5 (+); no longer R5.1, R6.1, R7.1, R8.1
- net A: now also J22.4 (Pin_4), R92.1; no longer J22.14 (Pin_14)
- net AB: now also J23.7 (Pin_7); no longer J23.6 (Pin_6)
- net ABC: now also J23.8 (Pin_8); no longer J23.7 (Pin_7)
- net ABCD: now also J23.10 (Pin_10); no longer J23.8 (Pin_8)
- net B: now also J23.6 (Pin_6), R102.1; no longer J22.12 (Pin_12)
- net C: now also J23.12 (Pin_12), R103.1; no longer J22.11 (Pin_11)
- net CD: now also J22.10 (Pin_10); no longer J23.12 (Pin_12)
- net CDA: now also J22.9 (Pin_9); no longer J23.10 (Pin_10)
- net D: now also J22.14 (Pin_14), R93.1; no longer J22.13 (Pin_13)
- net DA: now also J22.8 (Pin_8); no longer J22.6 (Pin_6)
- net ENCA_A: now also J22.6 (Pin_6), S1.A; no longer J22.3 (Pin_3)
- net ENCA_B: now also J22.5 (Pin_5), S1.B; no longer J22.4 (Pin_4)
- net ENCA_SW: now also J22.3 (Pin_3), R5.1, R104.2; no longer J22.5 (Pin_5)
- net ENCB_A: now also R96.2, S3.A; no longer R7.2
- net ENCB_B: now also J23.3 (Pin_3), R94.2, S3.B; no longer J23.5 (Pin_5), R5.2
- net ENCB_SW: now also J23.5 (Pin_5), R98.1, S3.3 (SW); no longer J23.3 (Pin_3)
- net ENCC_A: now also J23.15 (Pin_15), R97.2, S4.A; no longer J23.13 (Pin_13), R8.2
- net ENCC_B: now also R95.2, S4.B; no longer R6.2
- net ENCC_SW: now also J23.13 (Pin_13), R99.2, S4.3 (SW); no longer J23.15 (Pin_15)
- net ENCD_A: now also J22.12 (Pin_12), S2.A; no longer J22.9 (Pin_9)
- net ENCD_B: now also J22.11 (Pin_11), S2.B; no longer J22.10 (Pin_10)
- net ENCD_SW: now also J22.13 (Pin_13), R6.2, S2.3 (SW); no longer J22.8 (Pin_8)
- net GND: now also R5.2, R6.1, Q11.2 (E), Q2.2 (E), Q5.2 (E), Q8.2 (E), R98.2, R99.1, S1.C, S2.C, S3.C, S4.C
- net at D5.2 (A): now also Q3.2 (E); no longer Q3.3 (E)
- net at R15.2: now also Q3.3 (C); no longer Q3.2 (C)
- net at D8.2 (A): now also Q6.2 (E); no longer Q6.3 (E)
- net at R21.2: now also Q6.3 (C); no longer Q6.2 (C)
- net at D11.2 (A): now also Q9.2 (E); no longer Q9.3 (E)
- net at R27.2: now also Q9.3 (C); no longer Q9.2 (C)
- net at D14.2 (A): now also Q12.2 (E); no longer Q12.3 (E)
- net at R33.2: now also Q12.3 (C); no longer Q12.2 (C)
- net at D6.2 (A): now also Q4.2 (E); no longer Q4.3 (E)
- net at R16.2: now also Q4.3 (C); no longer Q4.2 (C)
- net at D9.2 (A): now also Q7.2 (E); no longer Q7.3 (E)
- net at R22.2: now also Q7.3 (C); no longer Q7.2 (C)
- net at D12.2 (A): now also Q10.2 (E); no longer Q10.3 (E)
- net at R28.2: now also Q10.3 (C); no longer Q10.2 (C)
- net at D15.2 (A): now also Q13.2 (E); no longer Q13.3 (E)
- net at R34.2: now also Q13.3 (C); no longer Q13.2 (C)
- net at D3.2 (A): now also Q1.2 (E); no longer Q1.3 (E)
- net at R10.2: now also Q1.3 (C); no longer Q1.2 (C)
- new net: R104.1, S1.3 (SW)
- new net: Q2.3 (C), R105.1, R131.1, R7.1
- new net: R131.2, S1.2 (-G)
- new net: R105.2, S1.4 (-B)
- new net: R7.2, S1.1 (-R)
- new net: Q8.1 (B), R102.2
- new net: Q8.3 (C), R100.1
- new net: R100.2, S3.1 (-R), S3.2 (-G), S3.4 (-B)
- new net: Q11.1 (B), R103.2
- new net: Q11.3 (C), R101.1
- new net: R101.2, S4.1 (-R), S4.2 (-G), S4.4 (-B)
- new net: Q5.1 (B), R93.2
- new net: Q5.3 (C), R8.1
- new net: R8.2, S2.1 (-R), S2.2 (-G), S2.4 (-B)
- new net: Q2.1 (B), R92.2
Other:
- note added: "can’t tie all anodes \nand all cathodes\ntogether"
- moved on the sheet: D11, D12, D14, D15, D3, D5, D6, D8, D9, J10, J11, J12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

Commit message: revised LED drivers for encoders, fixed code in various places
Parts:
- added R132, R135, R136: 15K, Resistor_SMD:R_0805_2012Metric_Pad1.15x1.40mm_HandSolder, symbol device:R_US
- added R133, R134, R137, R138, R139, R140: 270R, Resistor_SMD:R_0805_2012Metric_Pad1.15x1.40mm_HandSolder, symbol device:R_US
- R10, R15, R16, R21, R22, R27, R28, R33, R34: value 470R -> 1K
- R100, R101, R8: value 470R -> 390R
- R102, R103, R12, R13, R18, R19, R24, R25, R30, R31, R9, R93: value 4.7K -> 10K
- R105, R131: value 390R -> 270R
- R7: value 420R -> 390R
- R92: value 2.2K -> 10K
Connections:
- net +12V: now also S2.5 (+), S3.5 (+), S4.5 (+)
- net +3V3: no longer S2.5 (+), S3.5 (+), S4.5 (+)
- net ENCB_SW: now also R136.2; no longer S3.3 (SW)
- net ENCC_SW: now also R135.2; no longer S4.3 (SW)
- net ENCD_SW: now also R132.2; no longer S2.3 (SW)
- net at Q8.3 (C), R100.1: now also R137.1, R139.1
- net at R100.2, S3.1 (-R): no longer S3.2 (-G), S3.4 (-B)
- net at Q11.3 (C), R101.1: now also R138.1, R140.1
- net at R101.2, S4.1 (-R): no longer S4.2 (-G), S4.4 (-B)
- net at Q5.3 (C), R8.1: now also R133.1, R134.1
- net at R8.2, S2.1 (-R): no longer S2.2 (-G), S2.4 (-B)
- new net: R139.2, S3.2 (-G)
- new net: R136.1, S3.3 (SW)
- new net: R137.2, S3.4 (-B)
- new net: R140.2, S4.2 (-G)
- new net: R135.1, S4.3 (SW)
- new net: R138.2, S4.4 (-B)
- new net: R134.2, S2.2 (-G)
- new net: R132.1, S2.3 (SW)
- new net: R133.2, S2.4 (-B)
Other:
- note added: "can’t tie all anodes \nand all cathodes\ntogether!\n"
- note removed: "can’t tie all anodes \nand all cathodes\ntogether"
- moved on the sheet: Q11, Q5, Q8, R100, R101, R102, R103, R6, R8, R93, R98, R99
