File: hardware/bells-theorem/power.sch (KiCad schematic (older format))
At the start: 13 parts, among them J1 Conn_02x05_Odd_Even, U2 L7805, U3 L78L33_TO92

Commit message: take gerbers out of the repo, push latest updates
Parts:
- removed U2: L7805, Package_TO_SOT_THT:TO-92_Inline_Wide, symbol regulator_linear:L7805
- added U2: L78L05_TO92, Package_TO_SOT_THT:TO-92_Inline_Wide, symbol regulator_linear:L78L05_TO92
Connections:
- net +12V: now also U2.3 (VI)
- net +5V: now also U2.1 (VO)
- net GND: now also U2.2 (GND)
Changed lines of the file:
@@
-	1    0    0    -1
-$EndComp
-$Comp
-L power:PWR_FLAG #FLG03
-U 1 1 5B65E029
-P 4750 3250
-F 0 "#FLG03" H 4750 3345 50  0001 C CNN
-F 1 "PWR_FLAG" H 4750 3430 50  0000 C CNN
-F 2 "" H 4750 3250 50  0000 C CNN
-F 3 "" H 4750 3250 50  0000 C CNN
-	1    4750 3250
 	1    0    0    -1
 $EndComp
@@
 Wire Wire Line
 	4450 3250 4750 3250
-Connection ~ 4750 3250
 Wire Wire Line
 	4450 3550 4450 3600
@@
 	4250 2900 4450 2900
 Wire Wire Line
-	3650 3250 4450 3250
+	3650 3250 4000 3250
 Connection ~ 3650 3250
 $Comp
@@
 $EndComp
 $Comp
-L regulator_linear:L7805 U2
-U 1 1 5F8CF7D5
-P 3500 4450
-F 0 "U2" H 3500 4692 50  0000 C CNN
-F 1 "L7805" H 3500 4601 50  0000 C CNN
-F 2 "Package_TO_SOT_THT:TO-92_Inline_Wide" H 3525 4300 50  0001 L CIN
-F 3 "http://www.st.com/content/ccc/resource/technical/document/datasheet/41/4f/b3/b0/12/d4/47/88/CD00000444.pdf/files/CD00000444.pdf/jcr:content/translations/en.CD00000444.pdf" H 3500 4400 50  0001 C CNN
-	1    3500 4450
-	1    0    0    -1
-$EndComp
-$Comp
 L device:C_Small C1
 U 1 1 5F8D08CF
@@
 $EndComp
 Connection ~ 5200 4450
+$Comp
+L power:PWR_FLAG #FLG0101
+U 1 1 607C458A
+P 4000 3250
+F 0 "#FLG0101" H 4000 3325 50  0001 C CNN
+F 1 "PWR_FLAG" H 4000 3423 50  0000 C CNN
+F 2 "" H 4000 3250 50  0001 C CNN
+F 3 "~" H 4000 3250 50  0001 C CNN
+	1    4000 3250
+	1    0    0    -1
+$EndComp
+Connection ~ 4000 3250
+Wire Wire Line
+	4000 3250 4450 3250
+$Comp
+L regulator_linear:L78L05_TO92 U2
+U 1 1 60614A90
+P 3500 4450
+F 0 "U2" H 3500 4692 50  0000 C CNN
+F 1 "L78L05_TO92" H 3500 4601 50  0000 C CNN
+F 2 "Package_TO_SOT_THT:TO-92_Inline_Wide" H 3500 4675 50  0001 C CIN
+F 3 "http://www.st.com/content/ccc/resource/technical/document/datasheet/15/55/e5/aa/23/5b/43/fd/CD00000446.pdf/files/CD00000446.pdf/jcr:content/translations/en.CD00000446.pdf" H 3500 4400 50  0001 C CNN
+	1    3500 4450
+	1    0    0    -1
+$EndComp
 $EndSCHEMATC

Commit message: version 0.3, update for corrected LED drivers, other tweaks
Parts:
- D1, D2: value D_Schottky -> CDBM140-G
- L1, L2: value Ferrite_Bead_Small -> BLM21PG220SH1D
Changed lines of the file:
@@
 P 4100 2900
 F 0 "D1" H 4100 2684 50  0000 C CNN
-F 1 "D_Schottky" H 4100 2775 50  0000 C CNN
+F 1 "CDBM140-G" H 4100 2775 50  0000 C CNN
 F 2 "Diode_SMD:D_SMA-SMB_Universal_Handsoldering" H 4100 2900 50  0001 C CNN
 F 3 "" H 4100 2900 50  0001 C CNN
@@
 P 4100 3600
 F 0 "D2" H 4100 3816 50  0000 C CNN
-F 1 "D_Schottky" H 4100 3725 50  0000 C CNN
+F 1 "CDBM140-G" H 4100 3725 50  0000 C CNN
 F 2 "Diode_SMD:D_SMA-SMB_Universal_Handsoldering" H 4100 3600 50  0001 C CNN
 F 3 "" H 4100 3600 50  0001 C CNN
@@
 P 3700 2900
 F 0 "L1" V 3463 2900 50  0000 C CNN
-F 1 "Ferrite_Bead_Small" V 3554 2900 50  0000 C CNN
+F 1 "BLM21PG220SH1D" V 3554 2900 50  0000 C CNN
 F 2 "Inductor_SMD:L_0805_2012Metric_Pad1.15x1.40mm_HandSolder" V 3630 2900 50  0001 C CNN
 F 3 "" H 3700 2900 50  0001 C CNN
@@
 P 3700 3600
 F 0 "L2" V 3800 3600 50  0000 C CNN
-F 1 "Ferrite_Bead_Small" V 3900 3600 50  0000 C CNN
+F 1 "BLM21PG220SH1D" V 3900 3600 50  0000 C CNN
 F 2 "Inductor_SMD:L_0805_2012Metric_Pad1.15x1.40mm_HandSolder" V 3630 3600 50  0001 C CNN
 F 3 "" H 3700 3600 50  0001 C CNN
