File: hardware/bells-theorem/bells-venn.kicad_pcb (KiCad board)
At the start: 2 copper layers, 257.4 x 128.5 mm, 304 parts, among them J1 Conn_02x05_Odd_Even, J10 D, J11 C, J12 DA, J13 CD, J14 DAB, J15 CDA, J16 A, J17 B, J18 AB, J19 BC, J2 left, J20 ABC, J21 BCD, J22 left, J23 right, J3 right, J4 IN, J5 CVA, J6 CVB, J7 CVC, J8 CVD, J9 ABCD, Q11 2N3904, Q2 2N3904, Q5 2N3904, Q8 2N3904, U1 Teensy4.1, U10 TL074, U11 SN74LV1T34DBV, U12 MCP6004, U13 MCP6002-xSN, U2 R-78B5.0-2.0, U3 ADP150-3.3, U4 TL074, U5 TL074, U6 TL074, U7 TL072, U8 TL074, U9 TL074

Commit message: last hardware / software updates
Parts:
- removed C15, C17, C19, C21, C35, C37, C39: 100nF, Capacitor_SMD:C_0805_2012Metric_Pad1.18x1.45mm_HandSolder
- removed C5: 10uF, Capacitor_THT:CP_Radial_D5.0mm_P2.50mm
- removed D2: CDBM140-G, Diode_SMD:D_SMA-SMB_Universal_Handsoldering
- removed the G*** at (60.8, 58.3) (x2)
- removed L2: BLM21PG220SH1D, Inductor_SMD:L_0805_2012Metric_Pad1.15x1.40mm_HandSolder
- removed Q11, Q2, Q5, Q8: 2N3904, Package_TO_SOT_SMD:SOT-23_Handsoldering
- removed R101: 360R, Resistor_SMD:R_0805_2012Metric_Pad1.20x1.40mm_HandSolder
- removed R102, R103: 15K, Resistor_SMD:R_0805_2012Metric_Pad1.20x1.40mm_HandSolder
- removed R105, R131, R133, R134, R137, R138, R139, R140: 270R, Resistor_SMD:R_0805_2012Metric_Pad1.20x1.40mm_HandSolder
- removed the REF** at (219.7, 60.5)
- added ?: , , F.Cu at (211.3, 101.9)
- added ?: , , F.Cu at (227.7, 32.4)
- added ?: , , F.Cu at (219.0, 70.5)
- added ?: , , F.Cu at (211.9, 85.1)
- added C30: 100nF, Capacitor_SMD:C_0805_2012Metric_Pad1.18x1.45mm_HandSolder, B.Cu at (166.8, 46.4)
- added C31: 100nF, Capacitor_SMD:C_0805_2012Metric_Pad1.18x1.45mm_HandSolder, B.Cu at (174.6, 66.7)
- added C32: 100nF, Capacitor_SMD:C_0805_2012Metric_Pad1.18x1.45mm_HandSolder, B.Cu at (124.8, 62.8)
- added C34: 2n, Capacitor_SMD:C_0805_2012Metric_Pad1.18x1.45mm_HandSolder, B.Cu at (209.7, 36.2)
- added C54: 2n, Capacitor_SMD:C_0805_2012Metric_Pad1.18x1.45mm_HandSolder, B.Cu at (209.8, 70.4)
- added C55: 2n, Capacitor_SMD:C_0805_2012Metric_Pad1.18x1.45mm_HandSolder, B.Cu at (209.6, 54.2)
- added C56: 2n, Capacitor_SMD:C_0805_2012Metric_Pad1.18x1.45mm_HandSolder, B.Cu at (209.5, 64.6)
- added C57: 2n, Capacitor_SMD:C_0805_2012Metric_Pad1.18x1.45mm_HandSolder, B.Cu at (209.5, 46.6)
- added C58: 2n, Capacitor_SMD:C_0805_2012Metric_Pad1.18x1.45mm_HandSolder, B.Cu at (209.8, 80.9)
- added C59: 100nF, Capacitor_SMD:C_0805_2012Metric_Pad1.18x1.45mm_HandSolder, B.Cu at (247.5, 70.7)
- added C6: 100nF, Capacitor_SMD:C_0805_2012Metric_Pad1.18x1.45mm_HandSolder, B.Cu at (122.3, 53.3)
- added C60: 100nF, Capacitor_SMD:C_0805_2012Metric_Pad1.18x1.45mm_HandSolder, B.Cu at (226.9, 37.7)
- added C61: 10uF, Capacitor_THT:CP_Radial_D5.0mm_P2.50mm, B.Cu at (238.7, 130.2)
- added C62: 2n, Capacitor_SMD:C_0805_2012Metric_Pad1.18x1.45mm_HandSolder, B.Cu at (261.8, 89.9)
- added C63: 2n, Capacitor_SMD:C_0805_2012Metric_Pad1.18x1.45mm_HandSolder, B.Cu at (261.8, 62.0)
- added C64: 2n, Capacitor_SMD:C_0805_2012Metric_Pad1.18x1.45mm_HandSolder, B.Cu at (266.0, 39.3)
- added C65: 2n, Capacitor_SMD:C_0805_2012Metric_Pad1.18x1.45mm_HandSolder, B.Cu at (261.9, 46.2)
- added C66: 2n, Capacitor_SMD:C_0805_2012Metric_Pad1.18x1.45mm_HandSolder, B.Cu at (266.0, 55.3)
- added C67: 2n, Capacitor_SMD:C_0805_2012Metric_Pad1.18x1.45mm_HandSolder, B.Cu at (265.9, 83.1)
- added C68: 2n, Capacitor_SMD:C_0805_2012Metric_Pad1.18x1.45mm_HandSolder, B.Cu at (265.7, 71.4)
- added J24: 5V_SEL, Connector_PinHeader_2.54mm:PinHeader_1x03_P2.54mm_Vertical, B.Cu at (257.0, 132.1)
- added R19: 100R, Resistor_SMD:R_0805_2012Metric_Pad1.20x1.40mm_HandSolder, B.Cu at (122.4, 51.0)
- added R21: 100R, Resistor_SMD:R_0805_2012Metric_Pad1.20x1.40mm_HandSolder, B.Cu at (128.9, 62.8)
- added R22: 33R, Resistor_SMD:R_0805_2012Metric_Pad1.20x1.40mm_HandSolder, B.Cu at (144.1, 52.1)
- added R24: 33R, Resistor_SMD:R_0805_2012Metric_Pad1.20x1.40mm_HandSolder, B.Cu at (145.0, 77.2)
- added R25: 33R, Resistor_SMD:R_0805_2012Metric_Pad1.20x1.40mm_HandSolder, B.Cu at (144.2, 71.0)
- added R27: 33R, Resistor_SMD:R_0805_2012Metric_Pad1.20x1.40mm_HandSolder, B.Cu at (153.7, 54.8)
- added R28: 33R, Resistor_SMD:R_0805_2012Metric_Pad1.20x1.40mm_HandSolder, B.Cu at (153.7, 76.5)
- added R30: 33R, Resistor_SMD:R_0805_2012Metric_Pad1.20x1.40mm_HandSolder, B.Cu at (153.8, 39.7)
- added R31: 33R, Resistor_SMD:R_0805_2012Metric_Pad1.20x1.40mm_HandSolder, B.Cu at (163.3, 52.0)
- added R33: 33R, Resistor_SMD:R_0805_2012Metric_Pad1.20x1.40mm_HandSolder, B.Cu at (164.4, 65.3)
- added R34: 33R, Resistor_SMD:R_0805_2012Metric_Pad1.20x1.40mm_HandSolder, B.Cu at (169.6, 63.0)
- added U14: WS2811, Package_SO:SOIC-8_3.9x4.9mm_P1.27mm, B.Cu at (127.4, 47.8)
- added U15: WS2811, Package_SO:SOIC-8_3.9x4.9mm_P1.27mm, B.Cu at (124.0, 69.3)
- added U16: WS2811, Package_SO:SOIC-8_3.9x4.9mm_P1.27mm, B.Cu at (172.5, 47.7)
- added U17: WS2811, Package_SO:SOIC-8_3.9x4.9mm_P1.27mm, B.Cu at (169.7, 69.0)
- added U18: L78L10, Package_TO_SOT_THT:TO-92_Inline_Wide, B.Cu at (232.7, 130.0)
- C10, C11, C12, C13, C22, C23, C24, C25, C26, C27, C7, C8, C9: value 1nF -> 3.3n
- C2: value 1uF -> 1uF/10uF
- J1: value Conn_02x05_Odd_Even -> Euro_Power; footprint Connector_IDC:IDC-Header_2x05_P2.54mm_Vertical -> Connector_IDC:IDC-Header_2x08_P2.54mm_Vertical
- R100: value 360R -> 100R; moved to B.Cu
- R104, R132, R135, R136: value 15K -> 3.3K
- R119, R121, R16, R18: value 33K -> 47K
- R7, R8: value 360R -> 33R; moved to B.Cu
- R92: value 15K -> 100R; moved to B.Cu
- R93: value 15K -> 33R; moved to B.Cu
- moved R93 64.9 mm to (174.9, 53.5), turned to 0 degrees
- moved G*** 59.2 mm to (207.4, 112.0)
- moved R92 46.5 mm to (167.8, 49.3), turned to 0 degrees
- moved R8 42.5 mm to (135.5, 49.8), turned to -90 degrees
- moved R100 17.7 mm to (174.7, 62.6)
- moved REF** 13.9 mm to (119.3, 68.1)
- moved C2 10.8 mm to (254.3, 127.1), turned to 0 degrees
- moved R7 10.5 mm to (126.4, 53.0), turned to 180 degrees
- moved R9 4.93 mm to (122.6, 48.7), turned to 0 degrees
- moved REF** 3.61 mm to (215.4, 60.2)
- moved REF** 3.50 mm to (119.8, 53.5)
- moved ? 3.23 mm to (216.1, 95.1)
- moved REF** 2.68 mm to (161.5, 84.5)
- moved R59 2.05 mm to (265.9, 79.0)
- moved R50 2.05 mm to (265.9, 81.0)
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Connections:
- C14 pad 1: +12V -> +10V
- C16 pad 1: +12V -> +10V
- C18 pad 1: +12V -> +10V
- C20 pad 1: +12V -> +10V
- C28 pad 1: +12V -> +10V
- C36 pad 1: +12V -> +10V
- C38 pad 1: +12V -> +10V
- D11 pad 1: unconnected-(D11-Pad1) -> Net-(D11-Pad1)
- D11 pad 4: Net-(D10-Pad1) -> Net-(D11-Pad4)
- D4 pad 4: Net-(D3-Pad1) -> Net-(D4-Pad4)
- D5 pad 4: Net-(D4-Pad1) -> Net-(D5-Pad4)
- D7 pad 1: Net-(D6-Pad4) -> Net-(D7-Pad1)
- D8 pad 1: Net-(D7-Pad4) -> Net-(D8-Pad1)
- D8 pad 4: Net-(D5-Pad1) -> Net-(D8-Pad4)
- D9 pad 1: Net-(D10-Pad4) -> Net-(D9-Pad1)
- D9 pad 4: Net-(D6-Pad1) -> Net-(D9-Pad4)
- J2 pad 18: +12V -> +10V
- J22 pad 18: +12V -> +10V
- J4 pad 2: +12V -> +10V
- R100 pad 1: Net-(Q8-Pad3) -> +5V
- R100 pad 2: Net-(R100-Pad2) -> Net-(C31-Pad1)
- R119 pad 1: Net-(R119-Pad1) -> Net-(R116-Pad1)
- R119 pad 2: Net-(R116-Pad1) -> GND
- R120 pad 1: Net-(R120-Pad1) -> Net-(R118-Pad1)
- R120 pad 2: Net-(R118-Pad1) -> Net-(R120-Pad2)
- R121 pad 1: Net-(R121-Pad1) -> Net-(R117-Pad1)
- R121 pad 2: Net-(R117-Pad1) -> GND
- R128 pad 2: Net-(R119-Pad1) -> Net-(R128-Pad2)
- R129 pad 2: Net-(R121-Pad1) -> Net-(R129-Pad2)
- R130 pad 2: Net-(R120-Pad1) -> Net-(R120-Pad2)
- R16 pad 1: Net-(R114-Pad2) -> Net-(R13-Pad1)
- R16 pad 2: Net-(R13-Pad1) -> GND
- R18 pad 1: Net-(R115-Pad2) -> Net-(R15-Pad1)
- R18 pad 2: Net-(R15-Pad1) -> GND
- R7 pad 2: Net-(R7-Pad2) -> Net-(D3-Pad4)
- R8 pad 1: Net-(Q5-Pad3) -> Net-(D4-Pad4)
- R8 pad 2: Net-(R8-Pad2) -> Net-(D3-Pad1)
- R9 pad 2: Net-(D3-Pad4) -> Net-(R9-Pad2)
- R92 pad 1: /main/A -> +5V
- R93 pad 1: /main/D -> Net-(R93-Pad1)
- R93 pad 2: Net-(Q5-Pad1) -> Net-(D11-Pad1)
- S1 pad 1: Net-(R7-Pad2) -> Net-(S1-Pad1)
- S1 pad 5: +12V -> +5V
- S2 pad 1: Net-(R8-Pad2) -> Net-(S2-Pad1)
- S2 pad 5: +12V -> +5V
- S3 pad 1: Net-(R100-Pad2) -> Net-(S3-Pad1)
- S3 pad 5: +12V -> +5V
- S4 pad 5: +12V -> +5V
- U1 pad 15: unconnected-(U1-Pad15) -> Net-(C59-Pad2)
- U1 pad 46: unconnected-(U1-Pad46) -> Net-(C60-Pad1)
- U10 pad 11: -12V -> GND
- U10 pad 4: +12V -> +10V
- U12 pad 1: /main/scaleleft/scaleRef -> Net-(U12-Pad1)
- U12 pad 10: /main/scaleleft/scaleRef -> Net-(R117-Pad1)
- U12 pad 12: /main/scaleleft/scaleRef -> Net-(R116-Pad1)
- U12 pad 13: Net-(R116-Pad1) -> Net-(R128-Pad2)
- U12 pad 14: Net-(R119-Pad1) -> Net-(R128-Pad2)
- U12 pad 2: /main/scaleleft/scaleRef -> Net-(U12-Pad1)
- U12 pad 5: /main/scaleleft/scaleRef -> Net-(U12-Pad1)
- U12 pad 7: Net-(R120-Pad1) -> Net-(R120-Pad2)
- U12 pad 8: Net-(R121-Pad1) -> Net-(R129-Pad2)
- U12 pad 9: Net-(R117-Pad1) -> Net-(R129-Pad2)
- U13 pad 2: Net-(R13-Pad1) -> Net-(R114-Pad2)
- U13 pad 3: /main/scaleleft/scaleRef -> Net-(R13-Pad1)
- U13 pad 5: /main/scaleleft/scaleRef -> Net-(R15-Pad1)
- U13 pad 6: Net-(R15-Pad1) -> Net-(R115-Pad2)
- U2 pad 3: +5V -> Net-(J24-Pad1)
- U4 pad 11: -12V -> GND
- U4 pad 4: +12V -> +10V
- U5 pad 11: -12V -> GND
- U5 pad 4: +12V -> +10V
- U6 pad 11: -12V -> GND
- U6 pad 4: +12V -> +10V
- U7 pad 4: -12V -> GND
- U7 pad 8: +12V -> +10V
- U8 pad 11: -12V -> GND
- U8 pad 4: +12V -> +10V
- U9 pad 11: -12V -> GND
- U9 pad 4: +12V -> +10V
Routing:
- net +12V: track 478.2 -> 26.6 mm, vias 17 -> 0
- net +10V: track 0.00 -> 319.5 mm, vias 0 -> 14
- net -12V: track 239.1 -> 0.00 mm, vias 16 -> 0
- net +5V: track 390.8 -> 499.7 mm, vias 4 -> 7
- net /main/scaleleft/scaleRef: track 63.7 -> 0.00 mm, vias 2 -> 0
- net Net-(J1-Pad11): track 0.00 -> 42.2 mm
- net GND: track 126.2 -> 94.0 mm
- net Net-(R24-Pad2): track 0.00 -> 26.7 mm, vias 0 -> 2
- net Net-(R25-Pad1): track 0.00 -> 22.9 mm, vias 0 -> 2
- net Net-(S2-Pad1): track 0.00 -> 22.4 mm
- net Net-(D4-Pad1): track 21.8 -> 2.41 mm
- net Net-(S4-Pad1): track 3.74 -> 23.1 mm
- net Net-(D5-Pad4): track 0.00 -> 17.3 mm
- net Net-(J24-Pad1): track 0.00 -> 17.0 mm
- net /main/CVA: track 110.7 -> 94.2 mm
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Other:
- board text added: "-12V"
- board text added: "Bell’s Theorem prototype 0.5"
- board text added: "Copyright (c) 2022 Frogleg Synthesis"
- board text added: "DON'T FORGET TO REDO THE MASKS"
- board text added: "Options: - use 16 pin Euro header and take 5V from the rack. In this case omit the RECOM, C2 is 10uF - use 10 pin Euro Header and RECOM regulator for 5V. In this case add the RECOM, C2 is 1uF Jumper J24 to select"
- board text added: "P0"
- board text added: "P1"
- board text added: "P10"
- board text added: "P11"
- board text added: "P12"
- board text added: "P2"
- board text added: "P3"
- board text added: "P4"
- board text added: "P5"
- board text added: "P6"
- board text added: "P7"
- board text added: "P8"
- board text added: "P9"
- board text added: "This is pin 1 whether using 10 pin or 16 pin header"
- board text added: "This side for 5V from Recom"
- board text added: "This side for 5V rack power"
- board text removed: "Bell’s Theorem prototype 0.3"
- board text removed: "Bell’s Theorem prototype 0.4"
- board text removed: "Copyright (c) 2021 Frogleg Synthesis"
