File: hardware/bells-theorem/bells-venn.kicad_pcb (KiCad board)
At the start: 2 copper layers, 257.2 x 128.5 mm, 347 parts, among them J1 Euro_Power, J10 D, J11 C, J12 DA, J13 CD, J14 DAB, J15 CDA, J16 A, J17 B, J18 AB, J19 BC, J2 left, J20 ABC, J21 BCD, J22 left, J23 right, J24 5V_SEL, J3 right, J4 IN, J5 CVA, J6 CVB, J7 CVC, J8 CVD, J9 ABCD, U1 Teensy4.1, U10 TLV9304, U11 SN74LV1T34DBV, U12 MCP6004, U13 MCP6002-xSN, U14 WS2811, U15 WS2811, U16 WS2811, U17 WS2811, U18 L78L10, U19 TL071, U2 R-785.0-1.0, U3 ADP150-3.3, U4 TLV9304, U5 5, U6 TLV9304, U7 TLV9302, U8 TLV9304, U9 TLV9304

Commit message: checking in old outstanding changes prior to debugging with Claude Code
Parts:
- removed the ? at (235.8, 115.7)
- removed C61: 10uF, Capacitor_THT:CP_Radial_D5.0mm_P2.50mm
- removed the REF** at (258.6, 82.8)
- removed the REF** at (215.4, 60.2)
- removed RV1: 10K, myfootprints:pot_bourns_3296_dual-vertical
- removed U18: L78L10, Package_TO_SOT_THT:TO-92_Inline_Wide
- removed U19: TL071, Package_SO:SOIC-8_3.9x4.9mm_P1.27mm
- added ?: , , F.Cu at (227.8, 83.2)
- added ?: , , F.Cu at (223.7, 96.4)
- added ?: , , F.Cu at (248.9, 82.8)
- added ?: , , F.Cu at (226.4, 45.1)
- added ?: , , F.Cu at (226.6, 56.4)
- added R103: 30K, Resistor_SMD:R_0805_2012Metric_Pad1.20x1.40mm_HandSolder, B.Cu at (221.6, 58.3)
- added R105: 30K, Resistor_SMD:R_0805_2012Metric_Pad1.20x1.40mm_HandSolder, B.Cu at (221.6, 60.4)
- added R106: 30K, Resistor_SMD:R_0805_2012Metric_Pad1.20x1.40mm_HandSolder, B.Cu at (221.8, 76.9)
- added R107: 30K, Resistor_SMD:R_0805_2012Metric_Pad1.20x1.40mm_HandSolder, B.Cu at (221.9, 79.0)
- added R108: 10K, Resistor_SMD:R_0805_2012Metric_Pad1.20x1.40mm_HandSolder, B.Cu at (220.9, 37.3)
- added R109: 10K, Resistor_SMD:R_0805_2012Metric_Pad1.20x1.40mm_HandSolder, B.Cu at (220.9, 43.6)
- added R110: 10K, Resistor_SMD:R_0805_2012Metric_Pad1.20x1.40mm_HandSolder, B.Cu at (221.6, 56.3)
- added R111: 10K, Resistor_SMD:R_0805_2012Metric_Pad1.20x1.40mm_HandSolder, B.Cu at (221.6, 62.5)
- added R112: 10K, Resistor_SMD:R_0805_2012Metric_Pad1.20x1.40mm_HandSolder, B.Cu at (221.8, 74.7)
- added R113: 10K, Resistor_SMD:R_0805_2012Metric_Pad1.20x1.40mm_HandSolder, B.Cu at (221.9, 81.2)
- added R122: 30K, Resistor_SMD:R_0805_2012Metric_Pad1.20x1.40mm_HandSolder, B.Cu at (254.0, 35.7)
- added R123: 30K, Resistor_SMD:R_0805_2012Metric_Pad1.20x1.40mm_HandSolder, B.Cu at (254.0, 37.9)
- added R124: 30K, Resistor_SMD:R_0805_2012Metric_Pad1.20x1.40mm_HandSolder, B.Cu at (253.9, 54.5)
- added R125: 30K, Resistor_SMD:R_0805_2012Metric_Pad1.20x1.40mm_HandSolder, B.Cu at (253.9, 56.6)
- added R126: 30K, Resistor_SMD:R_0805_2012Metric_Pad1.20x1.40mm_HandSolder, B.Cu at (253.5, 85.0)
- added R127: 30K, Resistor_SMD:R_0805_2012Metric_Pad1.20x1.40mm_HandSolder, B.Cu at (253.5, 87.1)
- added R131: 30K, Resistor_SMD:R_0805_2012Metric_Pad1.20x1.40mm_HandSolder, B.Cu at (253.8, 74.3)
- added R133: 10K, Resistor_SMD:R_0805_2012Metric_Pad1.20x1.40mm_HandSolder, B.Cu at (254.0, 33.7)
- added R134: 10K, Resistor_SMD:R_0805_2012Metric_Pad1.20x1.40mm_HandSolder, B.Cu at (254.0, 39.9)
- added R137: 10K, Resistor_SMD:R_0805_2012Metric_Pad1.20x1.40mm_HandSolder, B.Cu at (253.9, 52.5)
- added R138: 10K, Resistor_SMD:R_0805_2012Metric_Pad1.20x1.40mm_HandSolder, B.Cu at (253.9, 58.6)
- added R139: 10K, Resistor_SMD:R_0805_2012Metric_Pad1.20x1.40mm_HandSolder, B.Cu at (253.5, 82.9)
- added R140: 10K, Resistor_SMD:R_0805_2012Metric_Pad1.20x1.40mm_HandSolder, B.Cu at (253.4, 89.1)
- added R141: 10K, Resistor_SMD:R_0805_2012Metric_Pad1.20x1.40mm_HandSolder, B.Cu at (262.1, 75.4)
- added R142: 300K, Resistor_SMD:R_0805_2012Metric_Pad1.20x1.40mm_HandSolder, B.Cu at (217.5, 90.0)
- added R143: 300K, Resistor_SMD:R_0805_2012Metric_Pad1.20x1.40mm_HandSolder, B.Cu at (211.1, 90.0)
- added R144: 100K, Resistor_SMD:R_0805_2012Metric_Pad1.20x1.40mm_HandSolder, B.Cu at (220.8, 89.8)
- added R145: 100K, Resistor_SMD:R_0805_2012Metric_Pad1.20x1.40mm_HandSolder, B.Cu at (207.2, 91.8)
- added R146: 300k, Resistor_SMD:R_0805_2012Metric_Pad1.20x1.40mm_HandSolder, B.Cu at (266.1, 105.1)
- added R147: 300k, Resistor_SMD:R_0805_2012Metric_Pad1.20x1.40mm_HandSolder, B.Cu at (253.5, 105.2)
- added R148: 100k, Resistor_SMD:R_0805_2012Metric_Pad1.20x1.40mm_HandSolder, B.Cu at (266.1, 103.0)
- added R149: 100k, Resistor_SMD:R_0805_2012Metric_Pad1.20x1.40mm_HandSolder, B.Cu at (253.6, 103.1)
- R10: value 20K -> 300K
- R101: value 10k -> 30K
- R102: value 4.7k -> 30K
- R116, R117, R118, R15: value 100K -> 300K
- R119, R121, R18: value 47K -> 100K
- R12: value 12K -> 100K
- R120: value 33K -> 100K
- R13: value 100K -> 300k
- R16: value 47K -> 100k
- moved R102 76.3 mm to (220.9, 41.6), turned to 0 degrees
- moved R101 68.4 mm to (220.9, 39.5)
- moved ? 33.4 mm to (249.0, 89.5)
- moved ? 27.4 mm to (251.9, 64.9)
- moved REF** 23.6 mm to (219.9, 75.8)
- moved REF** 22.5 mm to (212.2, 52.9)
- moved ? 19.4 mm to (214.7, 60.2)
- moved ? 16.7 mm to (269.1, 73.7)
- moved ? 16.7 mm to (247.7, 76.1)
- moved REF** 15.1 mm to (219.6, 57.3)
- moved REF** 14.5 mm to (249.7, 54.4)
- moved R12 14.4 mm to (215.5, 102.3), turned to -90 degrees
- moved REF** 14.2 mm to (225.4, 30.8)
- moved REF** 13.7 mm to (206.7, 64.0)
- moved REF** 13.5 mm to (270.3, 48.2)
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Connections:
- C14 pad 1: +10V -> +12V
- C15 pad 1: -10V -> -12V
- C16 pad 1: +10V -> +12V
- C17 pad 1: -10V -> -12V
- C18 pad 1: +10V -> +12V
- C19 pad 2: Net-(C19-Pad2) -> -12V
- C20 pad 1: +10V -> +12V
- C21 pad 1: -10V -> -12V
- C28 pad 1: +10V -> +12V
- C35 pad 1: -10V -> -12V
- C36 pad 1: +10V -> +12V
- C37 pad 1: -10V -> -12V
- C38 pad 1: +10V -> +12V
- C39 pad 1: -10V -> -12V
- C5 pad 1: -10V -> -12V
- C69 pad 1: Net-(C19-Pad2) -> -12V
- D2 pad 2: Net-(C19-Pad2) -> -12V
- J2 pad 18: +10V -> +5V
- J22 pad 18: +10V -> +5V
- J4 pad 2: +10V -> +5V
- R10 pad 1: +3V3 -> +5V
- R101 pad 1: +10V -> Net-(R101-Pad1)
- R101 pad 2: Net-(R101-Pad2) -> +5V
- R102 pad 1: Net-(R101-Pad2) -> Net-(R102-Pad1)
- R102 pad 2: Net-(R102-Pad2) -> +5V
- R116 pad 2: /main/CVB -> +5V
- R117 pad 2: /main/CVA -> +5V
- R13 pad 2: /main/CVC -> +5V
- R15 pad 2: /main/CVD -> +5V
- U10 pad 11: -10V -> -12V
- U10 pad 3: GND -> Net-(R106-Pad1)
- U10 pad 4: +10V -> +12V
- U10 pad 5: GND -> Net-(R107-Pad1)
- U12 pad 1: Net-(U12-Pad1) -> Net-(R120-Pad2)
- U12 pad 10: Net-(R117-Pad1) -> Net-(R116-Pad1)
- U12 pad 12: Net-(R116-Pad1) -> Net-(R117-Pad1)
- U12 pad 13: Net-(R128-Pad2) -> Net-(R142-Pad1)
- U12 pad 14: Net-(R128-Pad2) -> Net-(R129-Pad2)
- U12 pad 2: Net-(U12-Pad1) -> Net-(R118-Pad1)
- U12 pad 5: Net-(U12-Pad1) -> GND
- U12 pad 6: Net-(R118-Pad1) -> Net-(U12-Pad6)
- U12 pad 7: Net-(R120-Pad2) -> Net-(U12-Pad6)
- U12 pad 8: Net-(R129-Pad2) -> Net-(R128-Pad2)
- U12 pad 9: Net-(R129-Pad2) -> Net-(R143-Pad1)
- U13 pad 2: Net-(R114-Pad2) -> Net-(R146-Pad1)
- U13 pad 6: Net-(R115-Pad2) -> Net-(R147-Pad1)
- U4 pad 10: GND -> Net-(R123-Pad1)
- U4 pad 11: -10V -> -12V
- U4 pad 12: GND -> Net-(R122-Pad1)
- U4 pad 4: +10V -> +12V
- U5 pad 10: GND -> Net-(R125-Pad1)
- U5 pad 11: -10V -> -12V
- U5 pad 12: GND -> Net-(R124-Pad1)
- U5 pad 4: +10V -> +12V
- U6 pad 10: GND -> Net-(R127-Pad1)
- U6 pad 11: -10V -> -12V
- U6 pad 12: GND -> Net-(R126-Pad1)
- U6 pad 4: +10V -> +12V
- U7 pad 4: -10V -> -12V
- U7 pad 5: GND -> Net-(R131-Pad1)
- U7 pad 8: +10V -> +12V
- U8 pad 11: -10V -> -12V
- U8 pad 3: GND -> Net-(R101-Pad1)
- U8 pad 4: +10V -> +12V
- U8 pad 5: GND -> Net-(R102-Pad1)
- U9 pad 11: -10V -> -12V
- U9 pad 3: GND -> Net-(R103-Pad1)
- U9 pad 4: +10V -> +12V
- U9 pad 5: GND -> Net-(R105-Pad1)
Routing:
- net +10V: track 296.9 -> 0.00 mm, vias 16 -> 0
- net -12V: track 0.00 -> 277.3 mm, vias 0 -> 12
- net +5V: track 483.2 -> 748.6 mm, vias 14 -> 27
- net -10V: track 230.0 -> 0.00 mm, vias 15 -> 0
- net +12V: track 46.6 -> 265.3 mm, vias 1 -> 14
- net GND: track 116.2 -> 41.3 mm
- net Net-(C19-Pad2): track 36.8 -> 0.00 mm, vias 1 -> 0
- net /main/left outs/D_in: track 48.1 -> 22.9 mm, vias 3 -> 0
- net +3V3: track 295.7 -> 319.2 mm, vias 6 -> 10
- net /main/scaleleft/CVB_out: track 30.9 -> 46.6 mm, vias 1 -> 4
- net /main/np_ctl: track 60.0 -> 45.6 mm
- net /main/ENCB_SW: track 83.7 -> 71.5 mm, vias 2 -> 4
- net /main/scaleleft/CVA_out: track 37.8 -> 25.9 mm, vias 1 -> 2
- net Net-(R101-Pad2): track 12.0 -> 0.00 mm
- net /main/CVC: track 105.3 -> 116.5 mm, vias 2 -> 3
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Other:
- board text added: "Need to draw an even box around the ABCD jack to match the other outputs"
- board text removed: "-10V Adj"
- board text removed: "AAAAAAGH - main input scaling is wrong - consensus is accept -5V <> +5V rather than 0 - 10, on all inputs not just the {dblquote}input{dblquote} - Doing this isn't hard, but changes the supplies I'm using for normals ? - Except then do I need +/-10V for the op amps? Why not just distribute +/- 12V? Do I do bipolar output as well??"
- board text removed: "encb_sw"
- board text removed: "still a lot of silkscreen to clean up"
