File: hardware/bells-theorem/bells-venn.kicad_sch (KiCad schematic)
At the start: 0 parts

Commit message: All changes up to date with latest revisions
Other:
- sheet main ports: added 3Venable; removed none
- sheet power ports: added 3Venable; removed none
- title: Hexinverter Postman -> Bell's Theorem
